File: KiCAD-Project/STICKLEBACK.kicad_pcb (KiCad board)
At the start: 2 copper layers, 99.1 x 89.4 mm, 15 parts, among them J1 DE9_Pins_MountingHoles, J2 AudioJack3_SwitchTR, U1 74LS30, U2 74LS367, U3 74LS138

Commit message: Added PDF schematics
Other:
- board text added: "NOTE: PINS 9, 10, 13 NOT CONNECTED INTERNALLY IN 74LS30"
- board text added: "Rev 1.1 - Swapped R7 to C1 (10uF coupling capacitor) - Various silkscreen improvements - Some trace right angles removed - Some trace routing tidy-ups - Some minor via stitching"
- board text removed: "Rev 1.1 - Swapped R7 to C1 (10uF coupling capacitor) - Various silkscreen improvements - Some trace right angles removed - Some trace routing tidy-ups - Some minor Via stitching"
Changed lines of the file:
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@@
 	)
 	(paper "A4")
+	(title_block
+		(title "Stickleback")
+		(rev "1.1")
+		(company "Oddsocks b5s4")
+	)
 	(layers
 		(0 "F.Cu" signal)
@@
 		)
 	)
-	(gr_text "Rev 1.1\n- Swapped R7 to C1 (10uF coupling capacitor)\n- Various silkscreen improvements\n- Some trace right angles removed\n- Some trace routing tidy-ups\n- Some minor Via stitching\n"
+	(gr_text "NOTE: PINS 9, 10, 13 NOT CONNECTED INTERNALLY IN 74LS30"
+		(at 203.5 48 0)
+		(layer "User.1")
+		(effects
+			(font
+				(size 1 1)
+				(thickness 0.15)
+			)
+			(justify left bottom)
+		)
+	)
+	(gr_text "Rev 1.1\n- Swapped R7 to C1 (10uF coupling capacitor)\n- Various silkscreen improvements\n- Some trace right angles removed\n- Some trace routing tidy-ups\n- Some minor via stitching\n"
 		(at 203.2 60.96 0)
 		(layer "User.1")
